Commit message: gazebo and controller-package are not stable yet.

File: urdf/arm2r.urdf.xacro (robot description, xacro)
@@ -64,3 +64,23 @@
     <limit lower="-${pi}" upper="${pi}" effort="10" velocity="1.0"/>
   </joint>
+  <transmission name="${name}_tran1">
+    <type>transmission_interface/SimpleTransmission</type>
+    <robotNamespace>${name}</robotNamespace>
+    <joint name="joint_base_first">
+      <hardwareInterface>PositionJointInterface</hardwareInterface>
+    </joint>
+    <actuator name="${name}_motor1">
+      <mechanicalReduction>1</mechanicalReduction>
+    </actuator>
+  </transmission>
+  <transmission name="${name}_tran2">
+    <type>transmission_interface/SimpleTransmission</type>
+    <robotNamespace>${name}</robotNamespace>
+    <joint name="joint_first_second">
+      <hardwareInterface>PositionJointInterface</hardwareInterface>
+    </joint>
+    <actuator name="${name}_motor2">
+      <mechanicalReduction>1</mechanicalReduction>
+    </actuator>
+  </transmission>
 </robot>

Commit message: define {name}

File: urdf/arm2r.urdf.xacro (robot description, xacro)
@@ -4,4 +4,5 @@
   <xacro:property name="L2" value=".6" />
   <xacro:property name="pi" value="3.1415" />
+  <xacro:property name="name" value="arm2r" />
   <xacro:macro name="default_inertial" params="mass">
     <inertial>
